Commit message: Complete description of the robot and integration with gazebo

File: urdf/base.urdf.xacro (robot description, xacro)
@@ -32,4 +32,11 @@
     	</joint>
 		<link name="${name}_link">
+			<inertial>
+				<mass value="5"/>
+				<inertia
+					ixx="1" ixy="0.0" ixz="0.0"
+					iyy="1" iyz="0.0"
+					izz="1"/>
+			</inertial>
 			<visual>
 				<origin xyz="0 0 0" rpy="0 ${M_PI/2} ${M_PI/2}" />
@@ -50,4 +57,11 @@
 	<!-- Wheelchair Base - Link -->
 	<link name="base_link">
+		<inertial>
+			<mass value="100"/>
+			<inertia
+				ixx="1" ixy="0.0" ixz="0.0"
+				iyy="1" iyz="0.0"
+				izz="1"/>
+		</inertial>
 		<visual>
 			<origin xyz="${base_origin_x} ${base_origin_y} ${base_origin_z}" rpy="0 0 0"/>

File: urdf/seat.urdf.xacro (robot description, xacro)
@@ -43,4 +43,11 @@
     	</joint>
 		<link name="${name}_link">
+			<inertial>
+				<mass value="2"/>
+				<inertia
+					ixx="1e-6" ixy="0.0" ixz="0.0"
+					iyy="1e-6" iyz="0.0"
+					izz="1e-6"/>
+			</inertial>
 			<visual>
 				<origin xyz="0 0 0" rpy="0 0 0" />
@@ -70,4 +77,11 @@
 	<!-- Wheelchair Seat -->
 	<link name="seat_link">
+		<inertial>
+			<mass value="5"/>
+			<inertia
+				ixx="1e-6" ixy="0.0" ixz="0.0"
+				iyy="1e-6" iyz="0.0"
+				izz="1e-6"/>
+		</inertial>
 		<visual>
 			<geometry>
@@ -86,4 +100,11 @@
 	<!-- Wheelchair Back  -->
 	<link name="back_link">
+		<inertial>
+			<mass value="5"/>
+			<inertia
+				ixx="1e-6" ixy="0.0" ixz="0.0"
+				iyy="1e-6" iyz="0.0"
+				izz="1e-6"/>
+		</inertial>
 		<visual>
 			<geometry>

Commit message: New description of the wheelchair and the sensors

File: urdf/base.urdf.xacro (robot description, xacro)
@@ -3,24 +3,75 @@
 	<!-- Color are defined in materials.urdf.xacro -->
 	<xacro:property name="M_PI" value="3.1415926535897931" />
-	<xacro:property name="base_size_x"   value="0.63" />
-	<xacro:property name="base_size_y"   value="0.31" />
-	<xacro:property name="base_size_z"   value="0.30" />
-	<xacro:property name="base_origin_x" value="0.0" />
-	<xacro:property name="base_origin_y" value="0.0" />
-	<xacro:property name="base_origin_z" value="0.0" />
-	<xacro:property name="base_offset_z" value="0.078" />
-	<xacro:property name="wheel_main_radius"      value="0.175" />
-	<xacro:property name="wheel_main_width"       value="0.08" />
-	<xacro:property name="wheel_main_offset_x"    value="0.095" />
-	<xacro:property name="wheel_main_offset_y"    value="-0.295" />
+	<!-- Base origin and size -->
+	<xacro:property name="base_size_x"   value="0.462" />
+	<xacro:property name="base_size_y"   value="0.310" />
+	<xacro:property name="base_size_z"   value="0.270" />
+	<xacro:property name="base_origin_x" value="0.000" />
+	<xacro:property name="base_origin_y" value="0.000" />
+	<xacro:property name="base_origin_z" value="0.000" />
+	<xacro:property name="base_offset_z" value="0.073" />
+	<!-- Wheels size and offsets-->
+	<xacro:property name="wheel_main_radius"      value="0.167" />
+	<xacro:property name="wheel_main_width"       value="0.072" />
+	<xacro:property name="wheel_secondary_radius" value="0.070" />
+	<xacro:property name="wheel_secondary_width"  value="0.046" />
+	<xacro:property name="wheel_main_offset_x"    value="0.033" />
+	<xacro:property name="wheel_main_offset_y"    value="-0.278" />
 	<xacro:property name="wheel_main_offset_z"    value="${wheel_main_radius-base_offset_z-base_size_z/2}" />
-	<xacro:property name="wheel_secondary_radius" value="0.09" />
-	<xacro:property name="wheel_secondary_width"  value="0.04" />
-	<xacro:property name="wheel_front_offset_x"   value="0.385" />
-	<xacro:property name="wheel_front_offset_y"   value="-0.285" />
+	<xacro:property name="wheel_front_offset_x"   value="0.323" />
+	<xacro:property name="wheel_front_offset_y"   value="-0.257" />
 	<xacro:property name="wheel_front_offset_z"   value="${wheel_secondary_radius-base_offset_z-base_size_z/2}" />
-	<xacro:property name="wheel_back_offset_x"    value="-0.405" />
-	<xacro:property name="wheel_back_offset_y"    value="-0.225" />
+	<xacro:property name="wheel_back_offset_x"    value="-0.436" />
+	<xacro:property name="wheel_back_offset_y"    value="-0.187" />
 	<xacro:property name="wheel_back_offset_z"    value="${wheel_secondary_radius-base_offset_z-base_size_z/2}" />
+	<!-- Upper-base size and offset (related to base link)-->
+	<xacro:property name="upperbase_size_x" 	   value="0.491" />
+	<xacro:property name="upperbase_size_y" 	   value="0.247" />
+	<xacro:property name="upperbase_size_z" 	   value="0.040" />
+	<xacro:property name="upperbase_offset_x" 	   value="-0.063" />
+	<xacro:property name="upperbase_offset_y" 	   value="0.000" />
+	<xacro:property name="upperbase_offset_z" 	   value="0.199" />
+	<!-- Back structure size and offset (related to upperbase) -->
+	<xacro:property name="backstructure_size_x"		value="0.020" />
+	<xacro:property name="backstructure_size_y" 	value="0.460" />
+	<xacro:property name="backstructure_size_z" 	value="0.620" />
+	<xacro:property name="backstructure_offset_x"	value="-0.162" />
+	<xacro:property name="backstructure_offset_y"	value="0.000" />
+	<xacro:property name="backstructure_offset_z"	value="0.352" />
+	<!-- Armrest and offset (related to upperbase) -->
+	<xacro:property name="armrest_size_x"			value="0.278" />
+	<xacro:property name="armrest_size_y"			value="0.056" />
+	<xacro:property name="armrest_size_z"			value="0.036" />
+	<xacro:property name="armrest_offset_x"			value="0.068" />
+	<xacro:property name="armrest_offset_y"			value="-0.288" />
+	<xacro:property name="armrest_offset_z"			value="0.318" />
+	<!-- Bottomseat and offset (related to upperbase) -->
+	<xacro:property name="bottomseat_size_x"		value="0.440" />
+	<xacro:property name="bottomseat_size_y"		value="0.490" />
+	<xacro:property name="bottomseat_size_z"		value="0.130" />
+	<xacro:property name="bottomseat_offset_x"		value="0.109" />
+	<xacro:property name="bottomseat_offset_y"		value="0.000" />
+	<xacro:property name="bottomseat_offset_z"		value="0.151" />
+	<!-- Backseat and offset (related to upperbase) -->
+	<xacro:property name="backseat_size_x"			value="0.130" />
+	<xacro:property name="backseat_size_y"			value="0.460" />
+	<xacro:property name="backseat_size_z"			value="0.640" />
+	<xacro:property name="backseat_offset_x"		value="-0.047" />
+	<xacro:property name="backseat_offset_y"		value="0.000" />
+	<xacro:property name="backseat_offset_z"		value="0.502" />
+	<!-- Lowerplatform and offset (related to upperbase) -->
+	<xacro:property name="lowerplatform_size_x"		value="0.212" />
+	<xacro:property name="lowerplatform_size_y"		value="0.491" />
+	<xacro:property name="lowerplatform_size_z"		value="0.005" />
+	<xacro:property name="lowerplatform_offset_x"	value="-0.284" />
+	<xacro:property name="lowerplatform_offset_y"	value="0.000" />
+	<xacro:property name="lowerplatform_offset_z"	value="0.083" />
+	<!-- Upperplatform and offset (related to upperbase) -->
+	<xacro:property name="upperplatform_size_x"		value="0.310" />
+	<xacro:property name="upperplatform_size_y"		value="0.391" />
+	<xacro:property name="upperplatform_size_z"		value="0.010" />
+	<xacro:property name="upperplatform_offset_x"	value="-0.307" />
+	<xacro:property name="upperplatform_offset_y"	value="0.000" />
+	<xacro:property name="upperplatform_offset_z"	value="0.268" />
 <!-- ****************** Wheel macro ************************** -->
 	<xacro:macro name="wheel" params="name parent *shape *location">
@@ -55,5 +106,4 @@
 	</xacro:macro>
 <!-- ******************  Base ************************** -->
-	<!-- Wheelchair Base - Link -->
 	<link name="base_link">
 		<inertial>
@@ -75,4 +125,213 @@
 			<geometry>
 				<box size="${base_size_x} ${base_size_y} ${base_size_z}"/>
+			</geometry>
+		</collision>
+	</link>
+<!-- ******************  UpperBase ************************** -->
+	<joint name="upperbase_joint" type="prismatic">
+		<parent link="base_link"/>
+		<axis xyz="0 0 1"/>
+		<child link="upperbase_link"/>
+		<limit effort="1000.0" lower="0.0" upper="0.100" velocity="0.01"/>
+		<origin xyz="${upperbase_offset_x} ${upperbase_offset_y} ${upperbase_offset_z}"/>
+    </joint>
+	<link name="upperbase_link">
+		<inertial>
+			<mass value="10"/>
+			<inertia
+				ixx="1" ixy="0.0" ixz="0.0"
+				iyy="1" iyz="0.0"
+				izz="1"/>
+		</inertial>
+		<visual>
+			<geometry>
+				<box size="${upperbase_size_x} ${upperbase_size_y} ${upperbase_size_z}"/>
+			</geometry>
+			<material name="black"/>
+		</visual>
+		<collision>
+			<geometry>
+				<box size="${upperbase_size_x} ${upperbase_size_y} ${upperbase_size_z}"/>
+			</geometry>
+		</collision>
+	</link>
+<!-- ******************  BackStructure ************************** -->
+	<joint name="backstructure_joint" type="fixed">
+		<parent link="upperbase_link"/>
+		<child link="backstructure_link"/>
+		<origin xyz="${backstructure_offset_x} ${backstructure_offset_y} ${backstructure_offset_z}"/>
+    </joint>
+	<link name="backstructure_link">
+		<inertial>
+			<mass value="10"/>
+			<inertia
+				ixx="1" ixy="0.0" ixz="0.0"
+				iyy="1" iyz="0.0"
+				izz="1"/>
+		</inertial>
+		<visual>
+			<geometry>
+				<box size="${backstructure_size_x} ${backstructure_size_y} ${backstructure_size_z}"/>
+			</geometry>
+			<material name="black"/>
+		</visual>
+		<collision>
+			<geometry>
+				<box size="${backstructure_size_x} ${backstructure_size_y} ${backstructure_size_z}"/>
+			</geometry>
+		</collision>
+	</link>
+<!-- ******************  Bottomseat ************************** -->
+	<joint name="bottomseat_joint" type="fixed">
+		<parent link="upperbase_link"/>
+		<child link="bottomseat_link"/>
+		<origin xyz="${bottomseat_offset_x} ${bottomseat_offset_y} ${bottomseat_offset_z}"/>
+    </joint>
+	<link name="bottomseat_link">
+		<inertial>
+			<mass value="10"/>
+			<inertia
+				ixx="1" ixy="0.0" ixz="0.0"
+				iyy="1" iyz="0.0"
+				izz="1"/>
+		</inertial>
+		<visual>
+			<geometry>
+				<box size="${bottomseat_size_x} ${bottomseat_size_y} ${bottomseat_size_z}"/>
+			</geometry>
+			<material name="darkgrey"/>
+		</visual>
+		<collision>
+			<geometry>
+				<box size="${bottomseat_size_x} ${bottomseat_size_y} ${bottomseat_size_z}"/>
+			</geometry>
+		</collision>
+	</link>
+<!-- ******************  Backseat ************************** -->
+	<joint name="backseat_joint" type="fixed">
+		<parent link="upperbase_link"/>
+		<child link="backseat_link"/>
+		<origin xyz="${backseat_offset_x} ${backseat_offset_y} ${backseat_offset_z}"/>
+    </joint>
+	<link name="backseat_link">
+		<inertial>
+			<mass value="10"/>
+			<inertia
+				ixx="1" ixy="0.0" ixz="0.0"
+				iyy="1" iyz="0.0"
+				izz="1"/>
+		</inertial>
+		<visual>
+			<geometry>
+				<box size="${backseat_size_x} ${backseat_size_y} ${backseat_size_z}"/>
+			</geometry>
+			<material name="darkgrey"/>
+		</visual>
+		<collision>
+			<geometry>
+				<box size="${backseat_size_x} ${backseat_size_y} ${backseat_size_z}"/>
+			</geometry>
+		</collision>
+	</link>
+<!-- ******************  LowerPlatform ************************** -->
+	<joint name="lowerplatform_joint" type="fixed">
+		<parent link="upperbase_link"/>
+		<child link="lowerplatform_link"/>
+		<origin xyz="${lowerplatform_offset_x} ${lowerplatform_offset_y} ${lowerplatform_offset_z}"/>
+    </joint>
+	<link name="lowerplatform_link">
+		<inertial>
+			<mass value="10"/>
+			<inertia
+				ixx="1" ixy="0.0" ixz="0.0"
+				iyy="1" iyz="0.0"
+				izz="1"/>
+		</inertial>
+		<visual>
+			<geometry>
+				<box size="${lowerplatform_size_x} ${lowerplatform_size_y} ${lowerplatform_size_z}"/>
+			</geometry>
+			<material name="grey"/>
+		</visual>
+		<collision>
+			<geometry>
+				<box size="${lowerplatform_size_x} ${lowerplatform_size_y} ${lowerplatform_size_z}"/>
+			</geometry>
+		</collision>
+	</link>
+<!-- ******************  UpperPlatform ************************** -->
+	<joint name="upperplatform_joint" type="fixed">
+		<parent link="upperbase_link"/>
+		<child link="upperplatform_link"/>
+		<origin xyz="${upperplatform_offset_x} ${upperplatform_offset_y} ${upperplatform_offset_z}"/>
+    </joint>
+	<link name="upperplatform_link">
+		<inertial>
+			<mass value="10"/>
+			<inertia
+				ixx="1" ixy="0.0" ixz="0.0"
+				iyy="1" iyz="0.0"
+				izz="1"/>
+		</inertial>
+		<visual>
+			<geometry>
+				<box size="${upperplatform_size_x} ${upperplatform_size_y} ${upperplatform_size_z}"/>
+			</geometry>
+			<material name="grey"/>
+		</visual>
+		<collision>
+			<geometry>
+				<box size="${upperplatform_size_x} ${upperplatform_size_y} ${upperplatform_size_z}"/>
+			</geometry>
+		</collision>
+	</link>
+<!-- ******************  Armrests ************************** -->
+	<joint name="armrest_right_joint" type="fixed">
+		<parent link="upperbase_link"/>
+		<child link="armrest_right_link"/>
+		<origin xyz="${armrest_offset_x} ${armrest_offset_y} ${armrest_offset_z}"/>
+    </joint>
+	<link name="armrest_right_link">
+		<inertial>
+			<mass value="10"/>
+			<inertia
+				ixx="1" ixy="0.0" ixz="0.0"
+				iyy="1" iyz="0.0"
+				izz="1"/>
+		</inertial>
+		<visual>
+			<geometry>
+				<box size="${armrest_size_x} ${armrest_size_y} ${armrest_size_z}"/>
+			</geometry>
+			<material name="black"/>
+		</visual>
+		<collision>
+			<geometry>
+				<box size="${armrest_size_x} ${armrest_size_y} ${armrest_size_z}"/>
+			</geometry>
+		</collision>
+	</link>
+	<joint name="armrest_left_joint" type="fixed">
+		<parent link="upperbase_link"/>
+		<child link="armrest_left_link"/>
+		<origin xyz="${armrest_offset_x} ${-armrest_offset_y} ${armrest_offset_z}"/>
+    </joint>
+	<link name="armrest_left_link">
+		<inertial>
+			<mass value="10"/>
+			<inertia
+				ixx="1" ixy="0.0" ixz="0.0"
+				iyy="1" iyz="0.0"
+				izz="1"/>
+		</inertial>
+		<visual>
+			<geometry>
+				<box size="${armrest_size_x} ${armrest_size_y} ${armrest_size_z}"/>
+			</geometry>
+			<material name="black"/>
+		</visual>
+		<collision>
+			<geometry>
+				<box size="${armrest_size_x} ${armrest_size_y} ${armrest_size_z}"/>
 			</geometry>
 		</collision>

File: urdf/old/wheelchair.urdf.xacro (robot description, xacro)
@@ -5,4 +5,6 @@
 	<!-- Base urdf -->
 	<xacro:include filename="$(find cnbiros_wheelchair_description)/urdf/base.urdf.xacro" />
+	<!-- Upper part urdf -->
+	<xacro:include filename="$(find cnbiros_wheelchair_description)/urdf/seat.urdf.xacro" />
 	<!-- Sensors urdf -->
 	<xacro:include filename="$(find cnbiros_wheelchair_description)/urdf/sensors.urdf.xacro" />

File: urdf/sensors.urdf.xacro (robot description, xacro)
@@ -2,43 +2,47 @@
 <robot xmlns:xacro="http://www.ros.org/wiki/xacro" name="wheelchair">
 	<!-- Color are defined in materials.urdf.xacro -->
-	<xacro:property name="sonar_size_x"   value="0.012" />
-	<xacro:property name="sonar_size_y"   value="0.032" />
-	<xacro:property name="sonar_size_z"   value="0.015" />
-	<xacro:property name="sonar_0xe0_x"   value="0.19" />
-	<xacro:property name="sonar_0xe0_y"   value="-0.10" />
-	<xacro:property name="sonar_0xe0_z"   value="-0.05" />
-	<xacro:property name="sonar_0xe2_x"   value="0.450" />
-	<xacro:property name="sonar_0xe2_y"   value="-0.265" />
-	<xacro:property name="sonar_0xe2_z"   value="0.01" />
-	<xacro:property name="sonar_0xe4_x"   value="-0.165" />
-	<xacro:property name="sonar_0xe4_y"   value="-0.265" />
-	<xacro:property name="sonar_0xe4_z"   value="0.205" />
-	<xacro:property name="sonar_0xe6_x"   value="-0.513" />
-	<xacro:property name="sonar_0xe6_y"   value="-0.265" />
-	<xacro:property name="sonar_0xe6_z"   value="0.2455" />
-	<xacro:property name="sonar_0xe8_x"   value="-0.62" />
-	<xacro:property name="sonar_0xe8_y"   value="-0.238" />
-	<xacro:property name="sonar_0xe8_z"   value="0.3975" />
-	<xacro:property name="sonar_0xea_x"   value="0.19" />
-	<xacro:property name="sonar_0xea_y"   value="0.10" />
-	<xacro:property name="sonar_0xea_z"   value="-0.05" />
-	<xacro:property name="sonar_0xec_x"   value="0.450" />
-	<xacro:property name="sonar_0xec_y"   value="0.265" />
-	<xacro:property name="sonar_0xec_z"   value="0.01" />
-	<xacro:property name="sonar_0xee_x"   value="-0.165" />
-	<xacro:property name="sonar_0xee_y"   value="0.265" />
-	<xacro:property name="sonar_0xee_z"   value="0.205" />
-	<xacro:property name="sonar_0xf0_x"   value="-0.513" />
-	<xacro:property name="sonar_0xf0_y"   value="0.265" />
-	<xacro:property name="sonar_0xf0_z"   value="0.2455" />
-	<xacro:property name="sonar_0xf2_x"   value="-0.62" />
-	<xacro:property name="sonar_0xf2_y"   value="0.238" />
-	<xacro:property name="sonar_0xf2_z"   value="0.3975" />
-	<xacro:property name="kinect_size_x"   value="0.12" />
-	<xacro:property name="kinect_size_y"   value="0.32" />
-	<xacro:property name="kinect_size_z"   value="0.15" />
-	<xacro:property name="kinect_offset_x" value="0.15" />
-	<xacro:property name="kinect_offset_y" value="0.0" />
-	<xacro:property name="kinect_offset_z" value="0.2975" />
+	<!-- Ultrasonic sizes -->
+	<xacro:property name="sonar_size_x"		value="0.001" />
+	<xacro:property name="sonar_size_y"		value="0.032" />
+	<xacro:property name="sonar_size_z"		value="0.014" />
+	<!-- Kinect size -->
+	<xacro:property name="kinect_size_x"	value="0.061" />
+	<xacro:property name="kinect_size_y"	value="0.280" />
+	<xacro:property name="kinect_size_z"	value="0.038" />
+	<!-- Ultrasonic offset (with respect to base (e2, ec) or to upperbase) -->
+	<xacro:property name="sonar_0xe0_x"		value="0.324" />	<!-- TEMP -->
+	<xacro:property name="sonar_0xe0_y"   	value="-0.139" />	<!-- TEMP -->
+	<xacro:property name="sonar_0xe0_z"   	value="0.075" />	<!-- TEMP -->
+	<xacro:property name="sonar_0xe2_x"   	value="0.372" />	<!-- to base -->
+	<xacro:property name="sonar_0xe2_y"   	value="-0.257" />	<!-- to base -->
+	<xacro:property name="sonar_0xe2_z"   	value="0.048" />	<!-- to base -->
+	<xacro:property name="sonar_0xe4_x"   	value="0.168" />
+	<xacro:property name="sonar_0xe4_y"   	value="-0.240" />
+	<xacro:property name="sonar_0xe4_z"   	value="0.075" />
+	<xacro:property name="sonar_0xe6_x"   	value="-0.338" />
+	<xacro:property name="sonar_0xe6_y"   	value="-0.243" />
+	<xacro:property name="sonar_0xe6_z"   	value="0.080" />
+	<xacro:property name="sonar_0xe8_x"   	value="-0.458" />
+	<xacro:property name="sonar_0xe8_y"   	value="-0.126" />
+	<xacro:property name="sonar_0xe8_z"   	value="0.267" />
+	<xacro:property name="sonar_0xea_x"   	value="0.324" />	<!-- TEMP -->
+	<xacro:property name="sonar_0xea_y"   	value="0.139" />	<!-- TEMP -->
+	<xacro:property name="sonar_0xea_z"   	value="0.075" />	<!-- TEMP -->
+	<xacro:property name="sonar_0xec_x"   	value="0.372" />	<!-- to base -->
+	<xacro:property name="sonar_0xec_y"   	value="0.257" />	<!-- to base -->
+	<xacro:property name="sonar_0xec_z"   	value="0.048" />	<!-- to base -->
+	<xacro:property name="sonar_0xee_x"   	value="0.168" />
+	<xacro:property name="sonar_0xee_y"   	value="0.240" />
+	<xacro:property name="sonar_0xee_z"   	value="0.075" />
+	<xacro:property name="sonar_0xf0_x"   	value="-0.338" />
+	<xacro:property name="sonar_0xf0_y"   	value="0.243" />
+	<xacro:property name="sonar_0xf0_z"   	value="0.080" />
+	<xacro:property name="sonar_0xf2_x"   	value="-0.458" />
+	<xacro:property name="sonar_0xf2_y"   	value="0.136" />
+	<xacro:property name="sonar_0xf2_z"   	value="0.267" />
+	<!-- Kinect offset (with respect to upperbase) -->
+	<xacro:property name="kinect_offset_x"	value="0.294" />	<!-- TEMP -->
+	<xacro:property name="kinect_offset_y" 	value="0.000" />	<!-- TEMP -->
+	<xacro:property name="kinect_offset_z" 	value="0.002" />	<!-- TEMP -->
 <!-- ****************** Sonar macro ***************************** -->
 	<xacro:macro name="sonar" params="name parent *location">
@@ -71,5 +75,5 @@
 <!-- ****************** Sonars ***************************** -->
 	<!-- Sonar 0xe0 -->
-	<xacro:sonar name="sonar_0xe0" parent="base" >
+	<xacro:sonar name="sonar_0xe0" parent="upperbase" >
 		<origin xyz="${sonar_0xe0_x} ${sonar_0xe0_y} ${sonar_0xe0_z}" />
 	</xacro:sonar>
@@ -79,17 +83,17 @@
 	</xacro:sonar>
 	<!-- Sonar 0xe4 -->
-	<xacro:sonar name="sonar_0xe4" parent="base" >
+	<xacro:sonar name="sonar_0xe4" parent="upperbase" >
 		<origin xyz="${sonar_0xe4_x} ${sonar_0xe4_y} ${sonar_0xe4_z}" rpy="0 0 ${-M_PI/2}" />
 	</xacro:sonar>
 	<!-- Sonar 0xe6 -->
-	<xacro:sonar name="sonar_0xe6" parent="base" >
+	<xacro:sonar name="sonar_0xe6" parent="upperbase" >
 		<origin xyz="${sonar_0xe6_x} ${sonar_0xe6_y} ${sonar_0xe6_z}" rpy="0 0 ${-M_PI/2}"/>
 	</xacro:sonar>
 	<!-- Sonar 0xe8 -->
-	<xacro:sonar name="sonar_0xe8" parent="base" >
+	<xacro:sonar name="sonar_0xe8" parent="upperbase" >
 		<origin xyz="${sonar_0xe8_x} ${sonar_0xe8_y} ${sonar_0xe8_z}" rpy="0 0 ${-M_PI}"/>
 	</xacro:sonar>
 	<!-- Sonar 0xea -->
-	<xacro:sonar name="sonar_0xea" parent="base" >
+	<xacro:sonar name="sonar_0xea" parent="upperbase" >
 		<origin xyz="${sonar_0xea_x} ${sonar_0xea_y} ${sonar_0xea_z}" />
 	</xacro:sonar>
@@ -99,13 +103,13 @@
 	</xacro:sonar>
 	<!-- Sonar 0xee -->
-	<xacro:sonar name="sonar_0xee" parent="base" >
+	<xacro:sonar name="sonar_0xee" parent="upperbase" >
 		<origin xyz="${sonar_0xee_x} ${sonar_0xee_y} ${sonar_0xee_z}" rpy="0 0 ${M_PI/2}"/>
 	</xacro:sonar>
 	<!-- Sonar 0xf0 -->
-	<xacro:sonar name="sonar_0xf0" parent="base" >
+	<xacro:sonar name="sonar_0xf0" parent="upperbase" >
 		<origin xyz="${sonar_0xf0_x} ${sonar_0xf0_y} ${sonar_0xf0_z}" rpy="0 0 ${M_PI/2}"/>
 	</xacro:sonar>
 	<!-- Sonar 0xf2 -->
-	<xacro:sonar name="sonar_0xf2" parent="base" >
+	<xacro:sonar name="sonar_0xf2" parent="upperbase" >
 		<origin xyz="${sonar_0xf2_x} ${sonar_0xf2_y} ${sonar_0xf2_z}" rpy="0 0 ${-M_PI}"/>
 	</xacro:sonar>
@@ -134,5 +138,5 @@
 	<!-- Kinect - Joint -->
 	<joint name="camera_joint" type="fixed">
-		<parent link="base_link"/>
+		<parent link="upperbase_link"/>
 		<child link="camera_link"/>
 		<origin xyz="${kinect_offset_x} ${kinect_offset_y} ${kinect_offset_z}"/>
