Commit message: Updated the model of the wheelchair

File: urdf/base.urdf.xacro (robot description, xacro)
@@ -138,5 +138,5 @@
 	<link name="upperbase_link">
 		<inertial>
-			<mass value="10"/>
+			<mass value="50"/>
 			<inertia
 				ixx="1" ixy="0.0" ixz="0.0"
@@ -190,5 +190,5 @@
 	<link name="bottomseat_link">
 		<inertial>
-			<mass value="10"/>
+			<mass value="5"/>
 			<inertia
 				ixx="1" ixy="0.0" ixz="0.0"
@@ -216,5 +216,5 @@
 	<link name="backseat_link">
 		<inertial>
-			<mass value="10"/>
+			<mass value="1"/>
 			<inertia
 				ixx="1" ixy="0.0" ixz="0.0"
@@ -242,5 +242,5 @@
 	<link name="lowerplatform_link">
 		<inertial>
-			<mass value="10"/>
+			<mass value="1"/>
 			<inertia
 				ixx="1" ixy="0.0" ixz="0.0"
@@ -268,5 +268,5 @@
 	<link name="upperplatform_link">
 		<inertial>
-			<mass value="10"/>
+			<mass value="1"/>
 			<inertia
 				ixx="1" ixy="0.0" ixz="0.0"
@@ -294,5 +294,5 @@
 	<link name="armrest_right_link">
 		<inertial>
-			<mass value="10"/>
+			<mass value="0.5"/>
 			<inertia
 				ixx="1" ixy="0.0" ixz="0.0"
@@ -319,5 +319,5 @@
 	<link name="armrest_left_link">
 		<inertial>
-			<mass value="10"/>
+			<mass value="0.5"/>
 			<inertia
 				ixx="1" ixy="0.0" ixz="0.0"

File: urdf/sensors.urdf.xacro (robot description, xacro)
@@ -46,11 +46,11 @@
 	<xacro:property name="sonar_0xf2_z"   	value="0.267" />
 	<!-- Kinect offset (with respect to upperbase) -->
-	<xacro:property name="kinect_offset_x"	value="-0.365" /> <!-- !!! cyclope !!! -->
+	<xacro:property name="kinect_offset_x"	value="-0.430" /> <!-- !!! cyclope !!! -->
 	<xacro:property name="kinect_offset_y" 	value="0.000" />
-	<xacro:property name="kinect_offset_z" 	value="1.353" /> <!-- !!! Wheelchair's elevation !!! -->
+	<xacro:property name="kinect_offset_z" 	value="1.590" /> <!-- !!! Wheelchair's elevation !!! -->
 	<!-- Hokuyo offset (with respect to upperbase) -->
-	<xacro:property name="hokuyo_offset_x"	value="0.985" />
+	<xacro:property name="hokuyo_offset_x"	value="0.930" />
 	<xacro:property name="hokuyo_offset_y" 	value="0.000" />
-	<xacro:property name="hokuyo_offset_z" 	value="0.341" /> <!-- !!! Wheelchair's elevation !!! -->
+	<xacro:property name="hokuyo_offset_z" 	value="0.247" /> <!-- !!! Wheelchair's elevation !!! -->
 <!-- ****************** Sonar macro ***************************** -->
 	<xacro:macro name="sonar" params="name parent *location">
