Commit message: Added the collision for kinect

File: urdf/sensors.urdf.xacro (robot description, xacro)
@@ -126,4 +126,9 @@
 			<material name="green"/>
 		</visual>
+		<collision>
+			<geometry>
+				<box size="${kinect_size_x} ${kinect_size_y} ${kinect_size_z}" />
+			</geometry>
+		</collision>
 	</link>
 	<!-- Kinect - Joint -->

Commit message: Fixed the position of the kinect and the front ultrasonic sensors

File: urdf/sensors.urdf.xacro (robot description, xacro)
@@ -8,5 +8,5 @@
 	<xacro:property name="sonar_0xe0_y"   value="-0.10" />
 	<xacro:property name="sonar_0xe0_z"   value="-0.05" />
-	<xacro:property name="sonar_0xe2_x"   value="0.385" />
+	<xacro:property name="sonar_0xe2_x"   value="0.450" />
 	<xacro:property name="sonar_0xe2_y"   value="-0.265" />
 	<xacro:property name="sonar_0xe2_z"   value="0.01" />
@@ -23,5 +23,5 @@
 	<xacro:property name="sonar_0xea_y"   value="0.10" />
 	<xacro:property name="sonar_0xea_z"   value="-0.05" />
-	<xacro:property name="sonar_0xec_x"   value="0.385" />
+	<xacro:property name="sonar_0xec_x"   value="0.450" />
 	<xacro:property name="sonar_0xec_y"   value="0.265" />
 	<xacro:property name="sonar_0xec_z"   value="0.01" />
@@ -38,5 +38,5 @@
 	<xacro:property name="kinect_size_y"   value="0.32" />
 	<xacro:property name="kinect_size_z"   value="0.15" />
-	<xacro:property name="kinect_offset_x" value="0.565" />
+	<xacro:property name="kinect_offset_x" value="0.29" />
 	<xacro:property name="kinect_offset_y" value="0.0" />
 	<xacro:property name="kinect_offset_z" value="0.2975" />
@@ -76,5 +76,5 @@
 	<!-- Sonar 0xe2 -->
 	<xacro:sonar name="sonar_0xe2" parent="base" >
-		<origin xyz="${sonar_0xe2_x} ${sonar_0xe2_y} ${sonar_0xe2_z}" />
+		<origin xyz="${sonar_0xe2_x} ${sonar_0xe2_y} ${sonar_0xe2_z}" rpy="0 ${-M_PI/4} ${-M_PI/5}"/>
 	</xacro:sonar>
 	<!-- Sonar 0xe4 -->
@@ -96,5 +96,5 @@
 	<!-- Sonar 0xec -->
 	<xacro:sonar name="sonar_0xec" parent="base" >
-		<origin xyz="${sonar_0xec_x} ${sonar_0xec_y} ${sonar_0xec_z}" />
+		<origin xyz="${sonar_0xec_x} ${sonar_0xec_y} ${sonar_0xec_z}" rpy="0 ${-M_PI/4} ${M_PI/5}"/>
 	</xacro:sonar>
 	<!-- Sonar 0xee -->

Commit message: Modified kinect position

File: urdf/sensors.urdf.xacro (robot description, xacro)
@@ -5,5 +5,5 @@
 	<xacro:property name="sonar_size_y"   value="0.032" />
 	<xacro:property name="sonar_size_z"   value="0.015" />
-	<xacro:property name="sonar_0xe0_x"   value="0.365" />
+	<xacro:property name="sonar_0xe0_x"   value="0.19" />
 	<xacro:property name="sonar_0xe0_y"   value="-0.10" />
 	<xacro:property name="sonar_0xe0_z"   value="-0.05" />
@@ -20,5 +20,5 @@
 	<xacro:property name="sonar_0xe8_y"   value="-0.238" />
 	<xacro:property name="sonar_0xe8_z"   value="0.3975" />
-	<xacro:property name="sonar_0xea_x"   value="0.365" />
+	<xacro:property name="sonar_0xea_x"   value="0.19" />
 	<xacro:property name="sonar_0xea_y"   value="0.10" />
 	<xacro:property name="sonar_0xea_z"   value="-0.05" />
@@ -38,5 +38,5 @@
 	<xacro:property name="kinect_size_y"   value="0.32" />
 	<xacro:property name="kinect_size_z"   value="0.15" />
-	<xacro:property name="kinect_offset_x" value="0.29" />
+	<xacro:property name="kinect_offset_x" value="0.15" />
 	<xacro:property name="kinect_offset_y" value="0.0" />
 	<xacro:property name="kinect_offset_z" value="0.2975" />

Commit message: Modified the angle of the front sensors (e2 and ec) to pi/4

File: urdf/sensors.urdf.xacro (robot description, xacro)
@@ -80,5 +80,5 @@
 	<!-- Sonar 0xe2 -->
 	<xacro:sonar name="sonar_0xe2" parent="base" >
-		<origin xyz="${sonar_0xe2_x} ${sonar_0xe2_y} ${sonar_0xe2_z}" rpy="0 ${-M_PI/4} ${-M_PI/5}"/>
+		<origin xyz="${sonar_0xe2_x} ${sonar_0xe2_y} ${sonar_0xe2_z}" rpy="0 ${-M_PI/4} ${-M_PI/4}"/>
 	</xacro:sonar>
 	<!-- Sonar 0xe4 -->
@@ -100,5 +100,5 @@
 	<!-- Sonar 0xec -->
 	<xacro:sonar name="sonar_0xec" parent="base" >
-		<origin xyz="${sonar_0xec_x} ${sonar_0xec_y} ${sonar_0xec_z}" rpy="0 ${-M_PI/4} ${M_PI/5}"/>
+		<origin xyz="${sonar_0xec_x} ${sonar_0xec_y} ${sonar_0xec_z}" rpy="0 ${-M_PI/4} ${M_PI/4}"/>
 	</xacro:sonar>
 	<!-- Sonar 0xee -->

Commit message: Added hokuyo description to the wheelchair model

File: urdf/sensors.urdf.xacro (robot description, xacro)
@@ -10,4 +10,8 @@
 	<xacro:property name="kinect_size_y"	value="0.280" />
 	<xacro:property name="kinect_size_z"	value="0.038" />
+	<!-- Hokuyo size -->
+	<xacro:property name="hokuyo_size_x"	value="0.050" />
+	<xacro:property name="hokuyo_size_y"	value="0.050" />
+	<xacro:property name="hokuyo_size_z"	value="0.070" />
 	<!-- Ultrasonic offset (with respect to base (e2, ec) or to upperbase) -->
 	<xacro:property name="sonar_0xe0_x"		value="0.324" />	<!-- TEMP -->
@@ -44,5 +48,9 @@
 	<xacro:property name="kinect_offset_x"	value="0.294" />	<!-- TEMP -->
 	<xacro:property name="kinect_offset_y" 	value="0.000" />	<!-- TEMP -->
-	<xacro:property name="kinect_offset_z" 	value="0.002" />	<!-- TEMP -->
+	<xacro:property name="kinect_offset_z" 	value="0.105" />	<!-- TEMP -->
+	<!-- Hokuyo offset (with respect to upperbase) -->
+	<xacro:property name="hokuyo_offset_x"	value="0.272" />	<!-- TEMP -->
+	<xacro:property name="hokuyo_offset_y" 	value="0.000" />	<!-- TEMP -->
+	<xacro:property name="hokuyo_offset_z" 	value="0.035" />	<!-- TEMP -->
 <!-- ****************** Sonar macro ***************************** -->
 	<xacro:macro name="sonar" params="name parent *location">
@@ -142,3 +150,31 @@
 		<origin xyz="${kinect_offset_x} ${kinect_offset_y} ${kinect_offset_z}"/>
     </joint>
+<!-- ****************** Hokuyo ***************************** -->
+	<!-- Hokuyo - Link -->
+	<link name="hokuyo_link">
+		<inertial>
+			<mass value="0.5"/>
+			<inertia
+				ixx="1e-6" ixy="0.0" ixz="0.0"
+				iyy="1e-6" iyz="0.0"
+				izz="1e-6"/>
+		</inertial>
+		<visual>
+			<geometry>
+				<box size="${hokuyo_size_x} ${hokuyo_size_y} ${hokuyo_size_z}" />
+			</geometry>
+			<material name="green"/>
+		</visual>
+		<collision>
+			<geometry>
+				<box size="${hokuyo_size_x} ${hokuyo_size_y} ${hokuyo_size_z}" />
+			</geometry>
+		</collision>
+	</link>
+	<!-- Hokuyo - Joint -->
+	<joint name="hokuyo_joint" type="fixed">
+		<parent link="upperbase_link"/>
+		<child link="hokuyo_link"/>
+		<origin xyz="${hokuyo_offset_x} ${hokuyo_offset_y} ${hokuyo_offset_z}"/>
+    </joint>
 </robot>

Commit message: Updated the wheelchair description with the new support for laser and kinect

File: urdf/sensors.urdf.xacro (robot description, xacro)
@@ -46,11 +46,11 @@
 	<xacro:property name="sonar_0xf2_z"   	value="0.267" />
 	<!-- Kinect offset (with respect to upperbase) -->
-	<xacro:property name="kinect_offset_x"	value="0.294" />	<!-- TEMP -->
-	<xacro:property name="kinect_offset_y" 	value="0.000" />	<!-- TEMP -->
-	<xacro:property name="kinect_offset_z" 	value="0.105" />	<!-- TEMP -->
+	<xacro:property name="kinect_offset_x"	value="0.985" />
+	<xacro:property name="kinect_offset_y" 	value="0.000" />
+	<xacro:property name="kinect_offset_z" 	value="0.851" /> <!-- !!! Wheelchair's elevation !!! -->
 	<!-- Hokuyo offset (with respect to upperbase) -->
-	<xacro:property name="hokuyo_offset_x"	value="0.272" />	<!-- TEMP -->
-	<xacro:property name="hokuyo_offset_y" 	value="0.000" />	<!-- TEMP -->
-	<xacro:property name="hokuyo_offset_z" 	value="0.035" />	<!-- TEMP -->
+	<xacro:property name="hokuyo_offset_x"	value="0.985" />
+	<xacro:property name="hokuyo_offset_y" 	value="0.000" />
+	<xacro:property name="hokuyo_offset_z" 	value="0.341" /> <!-- !!! Wheelchair's elevation !!! -->
 <!-- ****************** Sonar macro ***************************** -->
 	<xacro:macro name="sonar" params="name parent *location">

Commit message: Commented the gazebo tag on kinect laser sensor (to reduce computational power). Switched back to gazebo laser plugin without gpu. Changed the resolution of the hokuyo laser to 120

File: urdf/sensors.urdf.xacro (robot description, xacro)
@@ -46,7 +46,7 @@
 	<xacro:property name="sonar_0xf2_z"   	value="0.267" />
 	<!-- Kinect offset (with respect to upperbase) -->
-	<xacro:property name="kinect_offset_x"	value="0.985" />
+	<xacro:property name="kinect_offset_x"	value="-0.365" /> <!-- !!! cyclope !!! -->
 	<xacro:property name="kinect_offset_y" 	value="0.000" />
-	<xacro:property name="kinect_offset_z" 	value="0.851" /> <!-- !!! Wheelchair's elevation !!! -->
+	<xacro:property name="kinect_offset_z" 	value="1.353" /> <!-- !!! Wheelchair's elevation !!! -->
 	<!-- Hokuyo offset (with respect to upperbase) -->
 	<xacro:property name="hokuyo_offset_x"	value="0.985" />
@@ -148,5 +148,5 @@
 		<parent link="upperbase_link"/>
 		<child link="camera_link"/>
-		<origin xyz="${kinect_offset_x} ${kinect_offset_y} ${kinect_offset_z}"/>
+		<origin xyz="${kinect_offset_x} ${kinect_offset_y} ${kinect_offset_z}" rpy="0 ${M_PI/9} 0"/>
     </joint>
 <!-- ****************** Hokuyo ***************************** -->

Commit message: Updated position of kinect (to be updated and re-checked)

File: urdf/sensors.urdf.xacro (robot description, xacro)
@@ -45,12 +45,12 @@
 	<xacro:property name="sonar_0xf2_y"   	value="0.136" />
 	<xacro:property name="sonar_0xf2_z"   	value="0.267" />
-	<!-- Kinect offset (with respect to upperbase) -->
-	<xacro:property name="kinect_offset_x"	value="-0.430" /> <!-- !!! cyclope !!! -->
+	<!-- Kinect offset (with respect to upperbase) - Cyclopic configuration -->
+	<xacro:property name="kinect_offset_x"	value="-0.20" /> <!-- !!! With respect to upperbase!!! -->
 	<xacro:property name="kinect_offset_y" 	value="0.000" />
-	<xacro:property name="kinect_offset_z" 	value="1.590" /> <!-- !!! Wheelchair's elevation !!! -->
+	<xacro:property name="kinect_offset_z" 	value="1.370" /> <!-- !!! With respect to upperbase!!! -->
 	<!-- Hokuyo offset (with respect to upperbase) -->
 	<xacro:property name="hokuyo_offset_x"	value="0.930" />
 	<xacro:property name="hokuyo_offset_y" 	value="0.000" />
-	<xacro:property name="hokuyo_offset_z" 	value="0.247" /> <!-- !!! Wheelchair's elevation !!! -->
+	<xacro:property name="hokuyo_offset_z" 	value="0.000" /> <!-- !!! With respect to upperbase!!! -->
 <!-- ****************** Sonar macro ***************************** -->
 	<xacro:macro name="sonar" params="name parent *location">
@@ -148,5 +148,5 @@
 		<parent link="upperbase_link"/>
 		<child link="camera_link"/>
-		<origin xyz="${kinect_offset_x} ${kinect_offset_y} ${kinect_offset_z}" rpy="0 ${M_PI/9} 0"/>
+		<origin xyz="${kinect_offset_x} ${kinect_offset_y} ${kinect_offset_z}" rpy="0 ${M_PI/6} 0"/>
     </joint>
 <!-- ****************** Hokuyo ***************************** -->
